File: Schematic_&_PCB/Duality.kicad_sch (KiCad schematic)
At the start: 0 parts

Commit message: continuing the pcb
Other:
- added sheet LEDs (LEDs.kicad_sch)
Changed lines of the file:
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@@
+		)
+	)
+	(sheet
+		(at 12.7 31.75)
+		(size 22.86 3.81)
+		(fields_autoplaced yes)
+		(stroke
+			(width 0.1524)
+			(type solid)
+		)
+		(fill
+			(color 0 0 0 0.0000)
+		)
+		(property "Sheetname" "LEDs"
+			(at 12.7 31.0384 0)
+			(effects
+				(font
+					(size 1.27 1.27)
+				)
+				(justify left bottom)
+			)
+		)
+		(property "Sheetfile" "LEDs.kicad_sch"
+			(at 12.7 36.1446 0)
+			(effects
+				(font
+					(size 1.27 1.27)
+				)
+				(justify left top)
+			)
+		)
+		(instances
+			(project "Duality"
+				(path "/ae9225e9-4453-4b68-a70e-f88602f2aa14"
+					(page "3")
+				)
+			)
 		)
 	)
