File: Schematic_&_PCB/LEDs.kicad_sch (KiCad schematic)
At the start: 166 parts

Commit message: I think i will change the MCU
Parts:
- renumbered C32 to C21, C33 to C22, C34 to C23, C35 to C24, C36 to C25, C37 to C26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
