File: Schematic_&_PCB/MatrixSwitch.kicad_sch (KiCad schematic)
At the start: 169 parts, among them SW1 ESC, SW10 F9, SW11 F10, SW12 F11, SW13 F12, SW14 `, SW15 1, SW16 2, SW17 3, SW18 4, SW19 5, SW2 F1, SW20 6, SW21 7, SW22 8, SW23 9, SW24 0, SW25 -, SW26 =, SW27 Backspace, SW28 Delete, SW29 Macro_1, SW3 F2, SW30 Macro_1, SW31 Macro_1, SW32 Macro_1, SW33 Macro_1, SW34 Macro_1, SW35 Macro_1, SW36 Macro_1, SW37 Macro_1, SW38 Macro_1, SW39 Macro_1, SW4 F3, SW40 Macro_1, SW41 Macro_1, SW42 Macro_1, SW43 Home, SW44 Macro_1, SW45 Macro_1, SW46 Macro_1, SW47 Macro_1, SW48 Macro_1, SW49 Macro_1, SW5 F4, SW50 Macro_1, SW51 Macro_1, SW52 Macro_1, SW53 Macro_1, SW54 Macro_1, SW55 Macro_1, SW56 Macro_1, SW57 Page Up, SW58 Macro_1, SW59 Macro_1, SW6 F5, SW60 Macro_1, SW61 Macro_1, SW62 Macro_1, SW63 Macro_1, SW64 Macro_1, SW65 Macro_1, SW66 Macro_1, SW67 Macro_1, SW68 Macro_1, SW69 Macro_1, SW7 F6, SW70 Macro_1, SW71 Page Down, SW72 Macro_1, SW73 Macro_1, SW74 Macro_1, SW75 Space, SW76 Space, SW77 Macro_1, SW78 Macro_1, SW79 Macro_1, SW8 F7, SW80 Macro_1, SW81 Macro_1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

Commit message: Started PCB
Parts:
- added D83: 1N4148WS, Diode_SMD:D_SOD-323, symbol Diode:1N4148WS
- added RE1: RotaryEncoder_Switch_MP, PCM_Miscellaneous:EC11E-Switch_Vertical_H11mm, symbol Device:RotaryEncoder_Switch_MP
- SW27: footprint PCM_Switch_Keyboard_Hotswap_Kailh:SW_Hotswap_Kailh_MX_Plated_1.00u -> PCM_Switch_Keyboard_Hotswap_Kailh:SW_Hotswap_Kailh_MX_Plated_2.00u
- SW29: value Macro_1 -> Tab; footprint PCM_Switch_Keyboard_Hotswap_Kailh:SW_Hotswap_Kailh_MX_Plated_1.00u -> PCM_Switch_Keyboard_Hotswap_Kailh:SW_Hotswap_Kailh_MX_Plated_1.50u
- SW30: value Macro_1 -> Q
- SW31: value Macro_1 -> W
- SW32: value Macro_1 -> E
- SW33: value Macro_1 -> R
- SW34: value Macro_1 -> T
- SW35: value Macro_1 -> Y
- SW36: value Macro_1 -> U
- SW37: value Macro_1 -> I
- SW38: value Macro_1 -> O
- SW39: value Macro_1 -> P
- SW40: value Macro_1 -> [
- SW41: value Macro_1 -> ]
- SW42: value Macro_1 -> \; footprint PCM_Switch_Keyboard_Hotswap_Kailh:SW_Hotswap_Kailh_MX_Plated_1.00u -> PCM_Switch_Keyboard_Hotswap_Kailh:SW_Hotswap_Kailh_MX_Plated_1.50u
- SW44: value Macro_1 -> Caps Lock; footprint PCM_Switch_Keyboard_Hotswap_Kailh:SW_Hotswap_Kailh_MX_Plated_1.00u -> PCM_Switch_Keyboard_Hotswap_Kailh:SW_Hotswap_Kailh_MX_Plated_1.25u
- SW45: value Macro_1 -> A
- SW46: value Macro_1 -> S
- SW47: value Macro_1 -> D
- SW48: value Macro_1 -> F
- SW49: value Macro_1 -> G
- SW50: value Macro_1 -> H
- SW51: value Macro_1 -> J
- SW52: value Macro_1 -> K
- SW53: value Macro_1 -> L
- SW54: value Macro_1 -> ;
- SW55: value Macro_1 -> '
- SW56: value Macro_1 -> Enter; footprint PCM_Switch_Keyboard_Hotswap_Kailh:SW_Hotswap_Kailh_MX_Plated_1.00u -> PCM_Switch_Keyboard_Hotswap_Kailh:SW_Hotswap_Kailh_MX_Plated_2.25u
- SW58: value Macro_1 -> Shift; footprint PCM_Switch_Keyboard_Hotswap_Kailh:SW_Hotswap_Kailh_MX_Plated_1.00u -> PCM_Switch_Keyboard_Hotswap_Kailh:SW_Hotswap_Kailh_MX_Plated_2.25u
- SW59: value Macro_1 -> Z
- SW60: value Macro_1 -> X
- SW61: value Macro_1 -> C
- SW62: value Macro_1 -> V
- SW63: value Macro_1 -> B
- SW64: value Macro_1 -> N
- SW65: value Macro_1 -> M
- SW66: value Macro_1 -> ,
- SW67: value Macro_1 -> .
- SW68: value Macro_1 -> /
- SW69: value Macro_1 -> Shift; footprint PCM_Switch_Keyboard_Hotswap_Kailh:SW_Hotswap_Kailh_MX_Plated_1.00u -> PCM_Switch_Keyboard_Hotswap_Kailh:SW_Hotswap_Kailh_MX_Plated_1.75u
- SW70: value Macro_1 -> ↑
- SW72: value Macro_1 -> Control; footprint PCM_Switch_Keyboard_Hotswap_Kailh:SW_Hotswap_Kailh_MX_Plated_1.00u -> PCM_Switch_Keyboard_Hotswap_Kailh:SW_Hotswap_Kailh_MX_Plated_1.25u
- SW73: value Macro_1 -> Windows; footprint PCM_Switch_Keyboard_Hotswap_Kailh:SW_Hotswap_Kailh_MX_Plated_1.00u -> PCM_Switch_Keyboard_Hotswap_Kailh:SW_Hotswap_Kailh_MX_Plated_1.25u
- SW74: value Macro_1 -> Alt; footprint PCM_Switch_Keyboard_Hotswap_Kailh:SW_Hotswap_Kailh_MX_Plated_1.00u -> PCM_Switch_Keyboard_Hotswap_Kailh:SW_Hotswap_Kailh_MX_Plated_1.25u
- SW75, SW76: footprint PCM_Switch_Keyboard_Hotswap_Kailh:SW_Hotswap_Kailh_MX_Plated_1.00u -> PCM_Switch_Keyboard_Hotswap_Kailh:SW_Hotswap_Kailh_MX_Plated_3.00u
- SW77: value Macro_1 -> Control
- SW78: value Macro_1 -> Alt
- SW79: value Macro_1 -> Menu
- SW80: value Macro_1 -> ←
- SW81: value Macro_1 -> ↓
- SW82: value Macro_1 -> →
Connections:
- net ROW1: now also D83.1 (K)
- net COL4: now reaches SW17.1 (A), SW3.1 (A), SW32.1 (A), SW47.1 (A), SW61.1 (A), SW75.1 (A)
- net COL6: now reaches SW19.1 (A), SW34.1 (A), SW49.1 (A), SW5.1 (A), SW63.1 (A)
- net COL10: now reaches SW23.1 (A), SW38.1 (A), SW53.1 (A), SW67.1 (A), SW77.1 (A), SW9.1 (A)
- net COL5: now reaches SW18.1 (A), SW33.1 (A), SW4.1 (A), SW48.1 (A), SW62.1 (A)
- net COL12: now reaches SW25.1 (A), SW40.1 (A), SW55.1 (A), SW79.1 (A)
- net COL12: now also SW10.1 (A); no longer SW11.1 (A), SW69.1 (A)
- net COL9: now reaches SW22.1 (A), SW37.1 (A), SW52.1 (A), SW66.1 (A), SW8.1 (A)
- net COL8: now reaches SW21.1 (A), SW36.1 (A), SW51.1 (A), SW65.1 (A), SW7.1 (A)
- net COL3: now reaches SW16.1 (A), SW2.1 (A), SW31.1 (A), SW46.1 (A), SW60.1 (A), SW74.1 (A)
- net COL15: now reaches SW28.1 (A), SW43.1 (A), SW57.1 (A), SW71.1 (A), SW82.1 (A)
- net COL15: now also SW13.1 (A)
- net COL1: now reaches SW1.1 (A), SW14.1 (A), SW29.1 (A), SW44.1 (A), SW58.1 (A), SW72.1 (A)
- net COL11: now reaches SW24.1 (A), SW39.1 (A), SW54.1 (A), SW68.1 (A), SW78.1 (A)
- net COL11: no longer SW10.1 (A)
- net COL14: now reaches SW27.1 (A), SW42.1 (A), SW70.1 (A), SW81.1 (A)
- net COL14: now also SW12.1 (A), SW56.1 (A); no longer SW13.1 (A)
- net COL2: now reaches SW15.1 (A), SW30.1 (A), SW45.1 (A), SW59.1 (A), SW73.1 (A)
- net COL2: now also RE1.S2
- net COL7: now reaches SW20.1 (A), SW35.1 (A), SW50.1 (A), SW6.1 (A), SW64.1 (A), SW76.1 (A)
- net COL13: now reaches SW26.1 (A), SW41.1 (A), SW80.1 (A)
- net COL13: now also SW11.1 (A), SW69.1 (A); no longer SW12.1 (A), SW56.1 (A)
- new net: D83.2 (A), RE1.S1
- new net GND: RE1.C, RE1.MP
- new net Rotary Encoder Pin A: RE1.A
- new net Rotary Encoder Pin B: RE1.B
Other:
- moved on the sheet: D1, D10, D11, D12, D13, D14, D15, D16, D17, D18, D19, D2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

Commit message: continuing the pcb
Parts:
- added D76: 1N4148WS, Diode_SMD:D_SOD-323, symbol Diode:1N4148WS
- added SW76: Space, PCM_Switch_Keyboard_Hotswap_Kailh:SW_Hotswap_Kailh_MX_Plated_6.25u, symbol Switch:SW_SPST
- renumbered D76 to D77, D77 to D78, D78 to D79, D79 to D80, D80 to D81, D81 to D82, D82 to D83, D83 to D84, SW76 to SW77, SW77 to SW78, SW78 to SW79, SW79 to SW80, SW80 to SW81, SW81 to SW82, SW82 to SW83
Connections:
- net COL6: now also SW76.1 (A)
- net COL7: no longer SW77.1 (A)
- net COL8: now also SW77.1 (A)
- net ROW6: now also D76.1 (K)
- new net: D76.2 (A), SW76.2 (B)
Other:
- moved on the sheet: D77, SW77
