File: Schematic_&_PCB/Microcontroller.kicad_sch (KiCad schematic)
At the start: 26 parts, among them J1 GCT USB4105, SW21 ~{RESET}, SW22 ~{USB_BOOT}, U1 RP2040, U2 W25Q32JVZP, U3 NCP1117ST33T3G, U4 USBLC6-2SC6, Y1 12MHz

Commit message: continuing the pcb
Parts:
- J1: value GCT USB4105 -> GCT USB45xx; footprint Connector_USB:USB_C_Receptacle_GCT_USB4105-xx-A_16P_TopMnt_Horizontal -> PCM_Miscellaneous:GCT_USB4505-03-0-A_REVA

Commit message: I think i will change the MCU
Parts:
- added U5: ATmega32U4-M, Package_DFN_QFN:QFN-44-1EP_7x7mm_P0.5mm_EP5.2x5.2mm, symbol MCU_Microchip_ATmega:ATmega32U4-M
- J1: footprint PCM_Miscellaneous:GCT_USB4505-03-0-A_REVA -> PCM_Miscellaneous:GCT_USB45xx
Connections:
- net GND: now also U5.15 (GND), U5.23 (GND), U5.35 (GND), U5.43 (GND), U5.45 (GND), U5.5 (UGND)
- new net: U5.14 (VCC), U5.34 (VCC)
- new net: U5.24 (AVCC), U5.44 (AVCC)
